Commit message: FA左臂完成封装ik的正逆运动学验证，并通过moveit & markerArray实现手掌位姿可视化

File: fa_moveit2_config/config/fa_robot.ros2_control.xacro (robot description, xacro)
@@ -106,4 +106,25 @@
                 <state_interface name="velocity"/>
             </joint>
+            <joint name="waist_yaw_joint">
+                <command_interface name="position"/>
+                <state_interface name="position">
+                  <param name="initial_value">${initial_positions['waist_yaw_joint']}</param>
+                </state_interface>
+                <state_interface name="velocity"/>
+            </joint>
+            <joint name="waist_roll_joint">
+                <command_interface name="position"/>
+                <state_interface name="position">
+                  <param name="initial_value">${initial_positions['waist_roll_joint']}</param>
+                </state_interface>
+                <state_interface name="velocity"/>
+            </joint>
+            <joint name="waist_pitch_joint">
+                <command_interface name="position"/>
+                <state_interface name="position">
+                  <param name="initial_value">${initial_positions['waist_pitch_joint']}</param>
+                </state_interface>
+                <state_interface name="velocity"/>
+            </joint>
         </ros2_control>
     </xacro:macro>

Commit message: 1. 增加功能:根据pelvis到地高度,计算双腿逆解,并支持mujoco可视化验证 2. 删除多余文件

File: fa_moveit2_config/config/fa_robot.ros2_control.xacro (robot description, xacro)
@@ -127,4 +127,88 @@
                 <state_interface name="velocity"/>
             </joint>
+            <joint name="left_hip_pitch_joint">
+                <command_interface name="position"/>
+                <state_interface name="position">
+                  <param name="initial_value">${initial_positions['left_hip_pitch_joint']}</param>
+                </state_interface>
+                <state_interface name="velocity"/>
+            </joint>
+            <joint name="left_hip_roll_joint">
+                <command_interface name="position"/>
+                <state_interface name="position">
+                  <param name="initial_value">${initial_positions['left_hip_roll_joint']}</param>
+                </state_interface>
+                <state_interface name="velocity"/>
+            </joint>
+            <joint name="left_hip_yaw_joint">
+                <command_interface name="position"/>
+                <state_interface name="position">
+                  <param name="initial_value">${initial_positions['left_hip_yaw_joint']}</param>
+                </state_interface>
+                <state_interface name="velocity"/>
+            </joint>
+            <joint name="left_knee_joint">
+                <command_interface name="position"/>
+                <state_interface name="position">
+                  <param name="initial_value">${initial_positions['left_knee_joint']}</param>
+                </state_interface>
+                <state_interface name="velocity"/>
+            </joint>
+            <joint name="left_ankle_pitch_joint">
+                <command_interface name="position"/>
+                <state_interface name="position">
+                  <param name="initial_value">${initial_positions['left_ankle_pitch_joint']}</param>
+                </state_interface>
+                <state_interface name="velocity"/>
+            </joint>
+            <joint name="left_ankle_roll_joint">
+                <command_interface name="position"/>
+                <state_interface name="position">
+                  <param name="initial_value">${initial_positions['left_ankle_roll_joint']}</param>
+                </state_interface>
+                <state_interface name="velocity"/>
+            </joint>
+            <joint name="right_hip_pitch_joint">
+                <command_interface name="position"/>
+                <state_interface name="position">
+                  <param name="initial_value">${initial_positions['right_hip_pitch_joint']}</param>
+                </state_interface>
+                <state_interface name="velocity"/>
+            </joint>
+            <joint name="right_hip_roll_joint">
+                <command_interface name="position"/>
+                <state_interface name="position">
+                  <param name="initial_value">${initial_positions['right_hip_roll_joint']}</param>
+                </state_interface>
+                <state_interface name="velocity"/>
+            </joint>
+            <joint name="right_hip_yaw_joint">
+                <command_interface name="position"/>
+                <state_interface name="position">
+                  <param name="initial_value">${initial_positions['right_hip_yaw_joint']}</param>
+                </state_interface>
+                <state_interface name="velocity"/>
+            </joint>
+            <joint name="right_knee_joint">
+                <command_interface name="position"/>
+                <state_interface name="position">
+                  <param name="initial_value">${initial_positions['right_knee_joint']}</param>
+                </state_interface>
+                <state_interface name="velocity"/>
+            </joint>
+            <joint name="right_ankle_pitch_joint">
+                <command_interface name="position"/>
+                <state_interface name="position">
+                  <param name="initial_value">${initial_positions['right_ankle_pitch_joint']}</param>
+                </state_interface>
+                <state_interface name="velocity"/>
+            </joint>
+            <joint name="right_ankle_roll_joint">
+                <command_interface name="position"/>
+                <state_interface name="position">
+                  <param name="initial_value">${initial_positions['right_ankle_roll_joint']}</param>
+                </state_interface>
+                <state_interface name="velocity"/>
+            </joint>
         </ros2_control>
     </xacro:macro>

File: sysmo_description/urdf/fa_robot.urdf (robot description, URDF)
Before this commit: robot fa_robot, 56 links, 55 joints
Links:
- removed link hand_base_link
- removed link index_distal
- removed link index_proximal
- removed link middle_distal
- removed link middle_proximal
- removed link pinky_distal
- removed link pinky_proximal
- removed link ring_distal
- removed link ring_proximal
- removed link thumb_distal
- removed link thumb_metacarpals
- removed link thumb_metacarpals_base2
- added link right_hand_base_link, mass 0.06740077960995; collision mesh filename=package://sysmo_description/meshes/right_hand_base_link.STL; visual mesh filename=package://sysmo_description/meshes/right_hand_base_link.STL
- added link right_index_distal, mass 0.00376787129082313; collision mesh filename=package://sysmo_description/meshes/right_index_distal.STL; visual mesh filename=package://sysmo_description/meshes/right_index_distal.STL
- added link right_index_proximal, mass 0.00253178529301663; collision mesh filename=package://sysmo_description/meshes/right_index_proximal.STL; visual mesh filename=package://sysmo_description/meshes/right_index_proximal.STL
- added link right_middle_distal, mass 0.00376786259758948; collision mesh filename=package://sysmo_description/meshes/right_middle_distal.STL; visual mesh filename=package://sysmo_description/meshes/right_middle_distal.STL
- added link right_middle_proximal, mass 0.00253175497594429; collision mesh filename=package://sysmo_description/meshes/right_middle_proximal.STL; visual mesh filename=package://sysmo_description/meshes/right_middle_proximal.STL
- added link right_pinky_distal, mass 0.00376782669873412; collision mesh filename=package://sysmo_description/meshes/right_pinky_distal.STL; visual mesh filename=package://sysmo_description/meshes/right_pinky_distal.STL
- added link right_pinky_proximal, mass 0.00253167400540778; collision mesh filename=package://sysmo_description/meshes/right_pinky_proximal.STL; visual mesh filename=package://sysmo_description/meshes/right_pinky_proximal.STL
- added link right_ring_distal, mass 0.0037678395356105; collision mesh filename=package://sysmo_description/meshes/right_ring_distal.STL; visual mesh filename=package://sysmo_description/meshes/right_ring_distal.STL
- added link right_ring_proximal, mass 0.00253170963529411; collision mesh filename=package://sysmo_description/meshes/right_ring_proximal.STL; visual mesh filename=package://sysmo_description/meshes/right_ring_proximal.STL
- added link right_thumb_distal, mass 0.00763302603723749; collision mesh filename=package://sysmo_description/meshes/right_thumb_distal.STL; visual mesh filename=package://sysmo_description/meshes/right_thumb_distal.STL
- added link right_thumb_metacarpals, mass 0.0123381607727595; collision mesh filename=package://sysmo_description/meshes/right_thumb_metacarpals.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; visual mesh filename=package://sysmo_description/meshes/right_thumb_metacarpals.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
- added link right_thumb_metacarpals_base2, mass 0.00138591070212997; collision mesh filename=package://sysmo_description/meshes/right_thumb_metacarpals_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; visual mesh filename=package://sysmo_description/meshes/right_thumb_metacarpals_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
Joints:
- removed joint index_dip
- removed joint index_mcp_pitch
- removed joint left_index_dip
- removed joint left_index_mcp_pitch
- removed joint left_middle_dip
- removed joint left_middle_mcp_pitch
- removed joint left_pinky_dip
- removed joint left_pinky_mcp_pitch
- removed joint left_ring_dip
- removed joint left_ring_mcp_pitch
- removed joint left_thumb_cmc_pitch
- removed joint left_thumb_cmc_yaw
- removed joint left_thumb_ip
- removed joint middle_dip
- removed joint middle_mcp_pitch
- removed joint pinky_dip
- removed joint pinky_mcp_pitch
- removed joint ring_dip
- removed joint ring_mcp_pitch
- removed joint thumb_cmc_pitch
- removed joint thumb_cmc_yaw
- removed joint thumb_ip
- added joint left_index_dip_joint: type revolute, parent left_index_proximal, child left_index_distal, origin xyz=-0.0052516 0 0.036625 rpy=0 0 0, axis 0 1 0, limit lower=0 upper=1.43 effort=100 velocity=1, mimic joint=left_index_mcp_pitch_joint multiplier=0.89 offset=0
- added joint left_index_mcp_pitch_joint: type revolute, parent left_hand_base_link, child left_index_proximal, origin xyz=0.0024758 -0.02419 0.098779 rpy=0.05236 0 0, axis 0 1 0, limit lower=0 upper=1.60 effort=100 velocity=1
- added joint left_middle_dip_joint: type revolute, parent left_middle_proximal, child left_middle_distal, origin xyz=-0.0052516 0 0.036625 rpy=0 0 0, axis 0 1 0, limit lower=0 upper=1.43 effort=100 velocity=1, mimic joint=left_middle_mcp_pitch_joint multiplier=0.89 offset=0
- added joint left_middle_mcp_pitch_joint: type revolute, parent left_hand_base_link, child left_middle_proximal, origin xyz=0.00052576 -0.00634 0.1027 rpy=0 0 0, axis 0 1 0, limit lower=0 upper=1.60 effort=100 velocity=1
- added joint left_pinky_dip_joint: type revolute, parent left_pinky_proximal, child left_pinky_distal, origin xyz=-0.0052516 0 0.036625 rpy=0 0 0, axis 0 1 0, limit lower=0 upper=1.43 effort=100 velocity=1, mimic joint=left_pinky_mcp_pitch_joint multiplier=0.89 offset=0
- added joint left_pinky_mcp_pitch_joint: type revolute, parent left_hand_base_link, child left_pinky_proximal, origin xyz=0.0024758 0.028372 0.092741 rpy=-0.087266 0 0, axis 0 1 0, limit lower=0 upper=1.60 effort=100 velocity=1
- added joint left_ring_dip_joint: type revolute, parent left_ring_proximal, child left_ring_distal, origin xyz=-0.0052516 0 0.036625 rpy=0 0 0, axis 0 1 0, limit lower=0 upper=1.43 effort=100 velocity=1, mimic joint=left_ring_mcp_pitch_joint multiplier=0.89 offset=0
- added joint left_ring_mcp_pitch_joint: type revolute, parent left_hand_base_link, child left_ring_proximal, origin xyz=0.0010258 0.011135 0.098767 rpy=-0.05236 0 0, axis 0 1 0, limit lower=0 upper=1.60 effort=100 velocity=1
- added joint left_thumb_cmc_pitch_joint: type revolute, parent left_thumb_metacarpals_base2, child left_thumb_metacarpals, origin xyz=0.0061649 -0.010678 -0.004891 rpy=0 -1.1529 2.0944, axis 0 1 0, limit lower=0 upper=0.58 effort=100 velocity=1
- added joint left_thumb_cmc_yaw_joint: type revolute, parent left_hand_base_link, child left_thumb_metacarpals_base2, origin xyz=0.011508 -0.022975 0.032794 rpy=0 0 0, axis 0 0 1, limit lower=0 upper=1.36 effort=100 velocity=1
- added joint left_thumb_ip_joint: type revolute, parent left_thumb_metacarpals, child left_thumb_distal, origin xyz=0.0037776 0 0.045368 rpy=0 0 0, axis 0 1 0, limit lower=0 upper=1.08 effort=100 velocity=1, mimic joint=left_thumb_cmc_pitch_joint multiplier=1.86 offset=0
- added joint right_index_dip_joint: type revolute, parent right_index_proximal, child right_index_distal, origin xyz=-0.0052516 0 0.036625 rpy=0 0 0, axis 0 1 0, limit lower=0 upper=1.43 effort=100 velocity=1, mimic joint=right_index_mcp_pitch_joint multiplier=0.89 offset=0
- added joint right_index_mcp_pitch_joint: type revolute, parent right_hand_base_link, child right_index_proximal, origin xyz=0.0024758 0.02419 0.098779 rpy=-0.05236 0 0, axis 0 1 0, limit lower=0 upper=1.60 effort=100 velocity=1
- added joint right_middle_dip_joint: type revolute, parent right_middle_proximal, child right_middle_distal, origin xyz=-0.0052516 0 0.036625 rpy=0 0 0, axis 0 1 0, limit lower=0 upper=1.43 effort=100 velocity=1, mimic joint=right_middle_mcp_pitch_joint multiplier=0.89 offset=0
- added joint right_middle_mcp_pitch_joint: type revolute, parent right_hand_base_link, child right_middle_proximal, origin xyz=0.00052576 0.00634 0.1027 rpy=0 0 0, axis 0 1 0, limit lower=0 upper=1.60 effort=100 velocity=1
- added joint right_pinky_dip_joint: type revolute, parent right_pinky_proximal, child right_pinky_distal, origin xyz=-0.0052516 0 0.036625 rpy=0 0 0, axis 0 1 0, limit lower=0 upper=1.43 effort=100 velocity=1, mimic joint=right_pinky_mcp_pitch_joint multiplier=0.89 offset=0
- added joint right_pinky_mcp_pitch_joint: type revolute, parent right_hand_base_link, child right_pinky_proximal, origin xyz=0.0024758 -0.028372 0.092741 rpy=0.087266 0 0, axis 0 1 0, limit lower=0 upper=1.60 effort=100 velocity=1
- added joint right_ring_dip_joint: type revolute, parent right_ring_proximal, child right_ring_distal, origin xyz=-0.0052516 0 0.036625 rpy=0 0 0, axis 0 1 0, limit lower=0 upper=1.43 effort=100 velocity=1, mimic joint=right_ring_mcp_pitch_joint multiplier=0.89 offset=0
- added joint right_ring_mcp_pitch_joint: type revolute, parent right_hand_base_link, child right_ring_proximal, origin xyz=0.0010258 -0.011135 0.098767 rpy=0.05236 0 0, axis 0 1 0, limit lower=0 upper=1.60 effort=100 velocity=1
- added joint right_thumb_cmc_pitch_joint: type revolute, parent right_thumb_metacarpals_base2, child right_thumb_metacarpals, origin xyz=0.0061649 0.010678 -0.004891 rpy=0 -1.1529 -2.0944, axis 0 1 0, limit lower=0 upper=0.58 effort=100 velocity=1
- added joint right_thumb_cmc_yaw_joint: type revolute, parent right_hand_base_link, child right_thumb_metacarpals_base2, origin xyz=0.011508 0.022975 0.032794 rpy=0 0 0, axis 0 0 -1, limit lower=0 upper=1.36 effort=100 velocity=1
- added joint right_thumb_ip_joint: type revolute, parent right_thumb_metacarpals, child right_thumb_distal, origin xyz=0.0037776 0 0.045368 rpy=0 0 0, axis 0 1 0, limit lower=0 upper=1.08 effort=100 velocity=1, mimic joint=right_thumb_cmc_pitch_joint multiplier=1.86 offset=0
- joint right_wrist_roll_jointfixed: child hand_base_link -> right_hand_base_link
