Commit message: v1.1.0: 轨迹优化支持FA neck，完成离线仿真自测

File: fa_moveit2_config/config/fa_robot.ros2_control.xacro (robot description, xacro)
@@ -211,4 +211,18 @@
                 <state_interface name="velocity"/>
             </joint>
+            <joint name="neck_yaw_joint">
+                <command_interface name="position"/>
+                <state_interface name="position">
+                  <param name="initial_value">${initial_positions['neck_yaw_joint']}</param>
+                </state_interface>
+                <state_interface name="velocity"/>
+            </joint>
+            <joint name="neck_pitch_joint">
+                <command_interface name="position"/>
+                <state_interface name="position">
+                  <param name="initial_value">${initial_positions['neck_pitch_joint']}</param>
+                </state_interface>
+                <state_interface name="velocity"/>
+            </joint>
         </ros2_control>
     </xacro:macro>
